File: hardware/v0.1.1/v0.1.1.kicad_pcb (KiCad board)
At the start: 2 copper layers, 110 x 70 mm, 31 parts

Commit message: added v0.1.1 to silk screen
Other:
- board text added: "Edge Computing Power Management Development Kit v0.1.1"
- board text removed: "Edge Computing Power Management Development Kit"
Changed lines of the file:
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@@
 		)
 	)
-	(gr_text "Edge Computing Power \nManagement Development Kit\n"
+	(gr_text "Edge Computing Power \nManagement Development Kit\nv0.1.1\n"
 		(at 212.5 143.4 0)
 		(layer "F.SilkS")
