File: hardware/v0.1.1/v0.1.1.kicad_pcb (KiCad board)
At the start: 2 copper layers, 110 x 70 mm, 31 parts

Commit message: Update references
Parts:
- PPG1: renamed from PPG Sensor
- RTC1: renamed from Real-time Clock
- VR1: renamed from Linear Regulator; value Voltage Regulator -> Linear Voltage Regulator
- renumbered Accelerometer to ACC1, Battery to B1, MicroSD to SD1, USB to USB1
Other:
- board text removed: "LR"
- board text removed: "MPU"
- board text removed: "MicroSD"

Commit message: Update pin electrical type MCU1
Parts:
- renumbered BT to BT1
Changed lines of the file:
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@@
 		(descr "Through hole straight pin header, 1x02, 2.00mm pitch, single row")
 		(tags "Through hole pin header THT 1x02 2.00mm single row")
-		(property "Reference" "BT"
+		(property "Reference" "BT1"
 			(at 0 5 180)
 			(layer "F.SilkS")
