File: hardware/v0.1.1/v0.1.1.kicad_sch (KiCad schematic)
At the start: 20 parts

Commit message: updates
Parts:
- renumbered USB2 to USB1

Commit message: Pin updates and power fixes
Parts:
- PPG1: symbol Connector:Conn_01x03_Female -> PATCH_sym_2:PPG_Connector
Other:
- moved on the sheet: C5, C6
