File: hardware/SPI NAND Flash Breakout Board/v0.1.0/SPI NAND Breakout.kicad_pcb (KiCad board)
At the start: 2 copper layers, 28 x 24.5 mm, 7 parts, among them J1 Conn_01x08_Pin, U1 AS5F18G04SND-10LIN

Commit message: updated schematic
Parts:
- removed U1: AS5F18G04SND-10LIN, AS5F18G04SND_10LIN:AS5F18G04SND-10LIN
- added C3: 100nF, Capacitor_SMD:C_0805_2012Metric, F.Cu at (156.3, 111.0)
- added C4: 100nF, Capacitor_SMD:C_0805_2012Metric, F.Cu at (156.3, 114.0)
- added C5: 1uF, Capacitor_SMD:C_0805_2012Metric, F.Cu at (156.3, 117.0)
- added C6: 100nF, Capacitor_SMD:C_0805_2012Metric, F.Cu at (156.3, 120.1)
- added R4: 10k, Resistor_SMD:R_0805_2012Metric, F.Cu at (160.7, 113.8)
- added U2: TXB0106PW, Package_SO:TSSOP-16_4.4x5mm_P0.65mm, F.Cu at (163.3, 118.6)
- added U3: AP2127K-1.8, Package_TO_SOT_SMD:SOT-23-5, F.Cu at (165.5, 105.9)
- C1: value 100nF -> 1uF; footprint Capacitor_SMD:C_0402_1005Metric -> Capacitor_SMD:C_0805_2012Metric
- C2: footprint Capacitor_SMD:C_0402_1005Metric -> Capacitor_SMD:C_0805_2012Metric
- R1, R2, R3: footprint Resistor_SMD:R_0402_1005Metric -> Resistor_SMD:R_0805_2012Metric
- moved C2 41.1 mm to (156.3, 108.0)
- moved J1 40.5 mm to (151.8, 105.8)
- moved C1 39.3 mm to (156.3, 105.0)
- moved R1 36.7 mm to (160.7, 105.0), turned to 0 degrees
- moved R3 31.9 mm to (160.7, 110.9)
- moved R2 31.0 mm to (160.7, 107.9)
Connections:
- C1 pad 1: Net-(J1-Pin_1) -> GND
- C1 pad 2: Net-(J1-Pin_8) -> Net-(J1-Pin_1)
- C2 pad 1: Net-(J1-Pin_1) -> GND
- C2 pad 2: Net-(J1-Pin_8) -> Net-(U1-VCC)
- J1 pad 8: Net-(J1-Pin_8) -> GND
- R1 pad 1: Net-(J1-Pin_1) -> Net-(U1-VCC)
- R1 pad 2: Net-(J1-Pin_2) -> Net-(U2-OE)
- R2 pad 1: Net-(J1-Pin_1) -> Net-(U1-CS#)
- R2 pad 2: Net-(J1-Pin_4) -> Net-(U1-VCC)
- R3 pad 1: Net-(J1-Pin_1) -> Net-(U1-VCC)
- R3 pad 2: Net-(J1-Pin_7) -> Net-(U1-WP#/SIO2)
Routing:
- net Net-(J1-Pin_1): track 6.73 -> 0.00 mm
Other:
- board outline removed

Commit message: Breakout Board Development
Parts:
- added U1: AS5F18G04SND-10LIN, Breakout:SON127P600X800X80-8N, F.Cu at (166.4, 97.0)
- moved C2 31.0 mm to (165.1, 78.3), turned to 180 degrees
- moved U2 28.2 mm to (161.9, 90.4), turned to 180 degrees
- moved C1 26.7 mm to (155.9, 78.3), turned to 180 degrees
- moved U3 25.5 mm to (160.0, 81.0)
- moved J1 25.3 mm to (152.0, 80.5)
- moved C3 8.60 mm to (161.3, 118.0)
- moved C4 8.60 mm to (161.3, 121.0)
- moved C5 8.60 mm to (161.3, 124.0)
- moved C6 8.60 mm to (161.3, 127.1)
- moved R1 8.60 mm to (165.7, 112.0)
- moved R2 8.60 mm to (165.7, 114.9)
- moved R3 8.60 mm to (165.7, 117.9)
- moved R4 8.60 mm to (165.7, 120.8)
Routing:
- net Net-(J1-Pin_1): track 0.00 -> 30.6 mm
- net Net-(J1-Pin_2): track 0.00 -> 14.6 mm, vias 0 -> 2
- net Net-(J1-Pin_7): track 0.00 -> 11.8 mm, vias 0 -> 1
- net Net-(J1-Pin_3): track 0.00 -> 11.5 mm, vias 0 -> 2
- net Net-(J1-Pin_6): track 0.00 -> 11.2 mm, vias 0 -> 2
- net Net-(J1-Pin_4): track 0.00 -> 8.75 mm, vias 0 -> 1
- net Net-(J1-Pin_5): track 0.00 -> 7.54 mm
- net GND: track 0.00 -> 6.73 mm, vias 0 -> 4
- net Net-(U1-VCC): track 0.00 -> 4.76 mm
- added copper zone on B.Cu, net GND
Other:
- board outline added: 32 x 24 mm

Commit message: gbr files
Parts:
- moved C6 36.4 mm to (170.2, 91.8), turned to 90 degrees
- moved R4 35.4 mm to (167.1, 85.5), turned to -90 degrees
- moved C5 32.9 mm to (167.7, 91.8), turned to 90 degrees
- moved C3 32.5 mm to (161.0, 85.5), turned to -90 degrees
- moved C4 26.9 mm to (156.2, 94.6), turned to 180 degrees
- moved R1 26.5 mm to (164.8, 85.5), turned to -90 degrees
- moved R3 20.6 mm to (156.2, 99.6)
- moved R2 20.0 mm to (156.2, 97.3), turned to 180 degrees
Routing:
- net Net-(U1-VCC): track 4.76 -> 54.9 mm, vias 0 -> 2
- net Net-(U1-HOLD#/SIO3): track 0.00 -> 18.3 mm
- net Net-(U1-WP#/SIO2): track 0.00 -> 17.7 mm, vias 0 -> 2
- net Net-(U1-SCLK): track 0.00 -> 13.6 mm, vias 0 -> 2
- net Net-(U1-CS#): track 0.00 -> 12.9 mm
- net Net-(U1-SI/SIO0): track 0.00 -> 12.8 mm, vias 0 -> 2
- net Net-(U1-SO/SIO1): track 0.00 -> 10.7 mm, vias 0 -> 2
- net Net-(J1-Pin_1): track 30.6 -> 35.1 mm, vias 0 -> 2
- net GND: track 6.73 -> 4.84 mm, vias 4 -> 31
- net Net-(U2-OE): track 0.00 -> 1.75 mm
- net Net-(J1-Pin_6): track 11.2 -> 10.2 mm
- added copper zone on F.Cu, net GND
Other:
- board size 32 x 24 mm -> 23.2 x 24 mm
- board text added: "3.3V"
- board text added: "CS#"
- board text added: "Flash: AS5F18G04SND-10LIN"
- board text added: "GND"
- board text added: "HOLD#/IO 3"
- board text added: "IO 0"
- board text added: "IO 1"
- board text added: "SCLK"
- board text added: "WP#/IO 2"

Commit message: more files
Parts:
- added G***: LOGO, LOGO, B.Cu at (169.5, 85.5)
