File: hardware/SPI NAND Flash Breakout Board/8 GBit/v0.1.0/SPI NAND Breakout.kicad_pcb (KiCad board)
At the start: 2 copper layers, 23.2 x 24 mm, 15 parts, among them J1 Conn_01x08_Pin, U1 AS5F18G04SND-10LIN, U2 TXB0106PW, U3 AP2127K-1.8

Commit message: text update
Other:
- board text added: "8 Gb"
- board text added: "v0.1.0"
Changed lines of the file:
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@@
 		(layer "Edge.Cuts")
 	)
-	(gr_text "Flash: AS5F18G04SND-10LIN"
+	(gr_text "8 Gb"
+		(at 171.997567 98.635127 0)
+		(layer "B.SilkS")
+		(effects
+			(font
+				(size 0.5 0.5)
+				(thickness 0.08)
+			)
+			(justify left bottom mirror)
+		)
+	)
+	(gr_text "v0.1.0"
 		(at 172 99.3 0)
 		(layer "B.SilkS")

Commit message: updated text
Other:
- board text added: "HOLD#/SIO3"
- board text added: "MISO/SIO1"
- board text added: "MOSI/SIO0"
- board text added: "SPI NAND: AS5F18G04SND-10LIN"
- board text added: "WP#/SIO2"
- board text removed: "Flash: AS5F18G04SND-10LIN"
- board text removed: "HOLD#/IO 3"
- board text removed: "IO 0"
- board text removed: "IO 1"
- board text removed: "WP#/IO 2"
Changed lines of the file:
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@@
 		)
 	)
-	(gr_text "Flash: AS5F18G04SND-10LIN"
+	(gr_text "SPI NAND: AS5F18G04SND-10LIN"
 		(at 172 100 0)
 		(layer "B.SilkS")
@@
 		)
 	)
-	(gr_text "CS#"
-		(at 157.939721 83.970852 0)
+	(gr_text "GND"
+		(at 157.832521 99.182322 0)
 		(layer "B.SilkS")
 		(effects
@@
 		)
 	)
-	(gr_text "GND"
-		(at 158.032521 99.182322 0)
-		(layer "B.SilkS")
-		(effects
-			(font
-				(size 1.5 1.5)
-				(thickness 0.3)
-				(bold yes)
-			)
-			(justify left bottom mirror)
-		)
-	)
-	(gr_text "IO 1"
-		(at 158.232521 86.482322 0)
-		(layer "B.SilkS")
-		(effects
-			(font
-				(size 1.5 1.5)
-				(thickness 0.3)
-				(bold yes)
-			)
-			(justify left bottom mirror)
-		)
-	)
-	(gr_text "IO 0"
-		(at 158.332521 91.582322 0)
+	(gr_text "CS#"
+		(at 157.839721 83.970852 0)
 		(layer "B.SilkS")
 		(effects
@@
 	)
 	(gr_text "3.3V"
-		(at 158.432521 81.482322 0)
+		(at 158.332521 81.482322 0)
 		(layer "B.SilkS")
 		(effects
@@
 	)
 	(gr_text "SCLK"
-		(at 159.032521 94.082322 0)
+		(at 158.932521 94.082322 0)
 		(layer "B.SilkS")
 		(effects
@@
 		)
 	)
-	(gr_text "WP#/IO 2"
-		(at 164.632521 88.982322 0)
+	(gr_text "HOLD#/SIO3"
+		(at 167.332521 96.682322 0)
 		(layer "B.SilkS")
 		(effects
@@
 		)
 	)
-	(gr_text "HOLD#/IO 3"
-		(at 167.232521 96.682322 0)
+	(gr_text "MISO/SIO1"
+		(at 153.032521 86.482322 0)
 		(layer "B.SilkS")
 		(effects
@@
 				(bold yes)
 			)
-			(justify left bottom mirror)
+			(justify right bottom mirror)
 		)
 	)
+	(gr_text "WP#/SIO2"
+		(at 153.032521 88.982322 0)
+		(layer "B.SilkS")
+		(effects
+			(font
+				(size 1.5 1.5)
+				(thickness 0.3)
+				(bold yes)
+			)
+			(justify right bottom mirror)
+		)
+	)
+	(gr_text "MOSI/SIO0"
+		(at 153.032521 91.582322 0)
+		(layer "B.SilkS")
+		(effects
+			(font
+				(size 1.5 1.5)
+				(thickness 0.3)
+				(bold yes)
+			)
+			(justify right bottom mirror)
+		)
+	)
